File: Solar Bauble - PCB/SolarBauble_v2 PCB.kicad_sch (KiCad schematic)
At the start: 27 parts, among them IC1 ATTINY85-P, P1 PCB_TEXT, P2 ISP, P4 HOLES, P5 LOGO1, P7 LOGO2, Q1 2N3906

Commit message: update on instructions
Other:
- title: Solar 8 Ball -> Solar Bauble
Changed lines of the file:
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@@
 	(paper "A4")
 	(title_block
-		(title "Solar 8 Ball")
-		(date "2020-04-07")
+		(title "Solar Bauble")
+		(date "2026-10-22")
 		(rev "1")
 		(company "The Curious Electric Compnay")
